File: WooferAmpIR2153.brd (EAGLE design)
At the start: 142.2 x 47.3 mm, 70 parts

Commit message: .
Parts:
- moved VD8 2.40 mm to (53.7, 14.3)
- moved R16 2.06 mm to (53.8, 16.5)
Routing:
- net N$2: track 24.5 -> 23.8 mm
Changed lines of the file:
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@@
 <setting verticaltext="up"/>
 </settings>
-<grid distance="6.25" unitdist="mil" unit="mil" style="lines" multiple="1" display="yes" altdistance="0.025" altunitdist="inch" altunit="inch"/>
+<grid distance="6.25" unitdist="mil" unit="mm" style="lines" multiple="1" display="yes" altdistance="0.025" altunitdist="inch" altunit="inch"/>
 <layers>
 <layer number="1" name="Top" color="4" fill="1" visible="yes" active="yes"/>
@@
 <attribute name="VALUE" x="50.4444" y="31.115" size="1.27" layer="28" ratio="10" rot="MR180"/>
 </element>
-<element name="R16" library="resistor" package="M1206" value="10" x="53.81625" y="14.44625" smashed="yes" rot="MR180">
-<attribute name="NAME" x="47.91075" y="15.77975" size="1.27" layer="26" ratio="10" rot="MR180"/>
-<attribute name="VALUE" x="49.33315" y="14.2875" size="1.27" layer="28" ratio="10" rot="MR180"/>
+<element name="R16" library="resistor" package="M1206" value="10" x="53.81625" y="16.51" smashed="yes" rot="MR180">
+<attribute name="NAME" x="47.91075" y="17.8435" size="1.27" layer="26" ratio="10" rot="MR180"/>
+<attribute name="VALUE" x="49.33315" y="16.35125" size="1.27" layer="28" ratio="10" rot="MR180"/>
 </element>
 <element name="R9" library="resistor" package="0207/10" value="3k3" x="36.5125" y="4.7625" smashed="yes">
@@
 <attribute name="VALUE" x="60.8965" y="35.90925" size="1.27" layer="28" ratio="10" rot="MR0"/>
 </element>
-<element name="VD8" library="diode" package="SOD80C" value="LL4148" x="53.975" y="16.66875" smashed="yes" rot="MR180">
-<attribute name="NAME" x="53.87975" y="23.33625" size="1.27" layer="26" ratio="10" rot="MR180"/>
-<attribute name="VALUE" x="52.29225" y="21.87575" size="1.27" layer="28" ratio="10" rot="MR180"/>
+<element name="VD8" library="diode" package="SOD80C" value="LL4148" x="53.6575" y="14.2875" smashed="yes" rot="MR180">
+<attribute name="NAME" x="53.56225" y="20.955" size="1.27" layer="26" ratio="10" rot="MR180"/>
+<attribute name="VALUE" x="51.97475" y="19.4945" size="1.27" layer="28" ratio="10" rot="MR180"/>
 </element>
 <element name="VT2" library="transistor" package="TO220V" value="13005" x="38.735" y="38.735" smashed="yes">
@@
 <wire x1="0.9525" y1="10.6375" x2="2.065" y2="9.525" width="1.6764" layer="16"/>
 <wire x1="48.895" y1="43.815" x2="48.895" y2="41.11625" width="1.778" layer="16"/>
-<wire x1="38.735" y1="39.0525" x2="32.7025" y2="39.0525" width="1.016" layer="16"/>
-<wire x1="38.735" y1="36.195" x2="38.735" y2="39.0525" width="1.016" layer="16"/>
-<wire x1="38.735" y1="39.0525" x2="42.545" y2="39.0525" width="1.016" layer="16"/>
-<wire x1="42.545" y1="39.0525" x2="43.815" y2="38.4175" width="1.016" layer="16"/>
-<wire x1="43.815" y1="38.4175" x2="46.0375" y2="38.4175" width="1.016" layer="16"/>
+<wire x1="38.735" y1="39.21125" x2="33.17875" y2="39.21125" width="1.016" layer="16"/>
+<wire x1="38.735" y1="36.195" x2="38.735" y2="39.21125" width="1.016" layer="16"/>
+<wire x1="38.735" y1="39.21125" x2="43.02125" y2="39.21125" width="1.016" layer="16"/>
+<wire x1="43.02125" y1="39.21125" x2="43.97375" y2="38.4175" width="1.016" layer="16"/>
+<wire x1="43.97375" y1="38.4175" x2="46.0375" y2="38.4175" width="1.016" layer="16"/>
 <wire x1="51.865" y1="43.7025" x2="54.2925" y2="43.815" width="1.016" layer="16"/>
 <contactref element="C21" pad="2"/>
@@
 <wire x1="26.3525" y1="18.57375" x2="27.14625" y2="19.3675" width="1.016" layer="16"/>
 <wire x1="32.0675" y1="43.4975" x2="32.0675" y2="43.815" width="1.27" layer="16"/>
-<wire x1="32.7025" y1="39.0525" x2="30.1625" y2="37.7825" width="1.016" layer="16"/>
+<wire x1="33.17875" y1="39.21125" x2="30.1625" y2="37.7825" width="1.016" layer="16"/>
 <wire x1="30.1625" y1="37.7825" x2="24.13" y2="37.7825" width="1.016" layer="16"/>
 <wire x1="24.13" y1="37.7825" x2="23.1775" y2="36.83" width="1.016" layer="16"/>
@@
 <contactref element="R16" pad="1"/>
 <contactref element="VD8" pad="C"/>
-<wire x1="52.41625" y1="14.44625" x2="52.275" y2="16.66875" width="1.016" layer="16"/>
-<wire x1="52.451" y1="10.795" x2="52.41625" y2="14.44625" width="1.016" layer="16"/>
 <wire x1="55.5625" y1="5.3975" x2="53.6575" y2="5.3975" width="1.016" layer="16"/>
 <wire x1="53.6575" y1="5.3975" x2="52.1335" y2="6.9215" width="1.016" layer="16"/>
 <wire x1="52.1335" y1="6.9215" x2="52.451" y2="10.795" width="1.016" layer="16"/>
+<wire x1="52.451" y1="10.795" x2="51.9575" y2="14.2875" width="1.016" layer="16"/>
+<wire x1="51.9575" y1="14.2875" x2="52.41625" y2="16.51" width="1.016" layer="16"/>
 </signal>
 <signal name="N$15">
@@
 <contactref element="R18" pad="2"/>
 <contactref element="VD8" pad="A"/>
-<wire x1="55.21625" y1="14.44625" x2="55.675" y2="16.66875" width="1.016" layer="16"/>
-<wire x1="55.21625" y1="14.44625" x2="55.08625" y2="12.35375" width="1.016" layer="16"/>
-<wire x1="58.42" y1="13.6525" x2="55.21625" y2="14.44625" width="1.016" layer="16"/>
+<wire x1="55.08625" y1="12.35375" x2="55.3575" y2="14.2875" width="1.016" layer="16"/>
+<wire x1="58.42" y1="13.6525" x2="55.3575" y2="14.2875" width="1.016" layer="16"/>
+<wire x1="55.3575" y1="14.2875" x2="55.21625" y2="16.51" width="1.016" layer="16"/>
 </signal>
 <signal name="GATE_A">
@@
 <contactref element="R17" pad="1"/>
 <wire x1="43.18" y1="12.7" x2="44.7675" y2="12.7" width="1.016" layer="16"/>
-<wire x1="44.7675" y1="12.7" x2="46.355" y2="14.2875" width="1.016" layer="16"/>
-<wire x1="46.355" y1="14.2875" x2="48.5775" y2="14.2875" width="1.016" layer="16"/>
-<wire x1="48.5775" y1="14.2875" x2="49.53" y2="15.24" width="1.016" layer="16"/>
+<wire x1="44.7675" y1="12.7" x2="46.51375" y2="14.44625" width="1.016" layer="16"/>
+<wire x1="46.51375" y1="14.44625" x2="48.73625" y2="14.44625" width="1.016" layer="16"/>
+<wire x1="48.73625" y1="14.44625" x2="49.53" y2="15.24" width="1.016" layer="16"/>
 <wire x1="49.53" y1="15.24" x2="49.53" y2="17.145" width="1.016" layer="16"/>
 <contactref element="U$4" pad="P$1"/>
@@
 <contactref element="R12" pad="2"/>
 <contactref element="VD4" pad="C"/>
-<wire x1="38.735" y1="32.7025" x2="37.1475" y2="33.02" width="1.016" layer="16"/>
-<wire x1="37.1475" y1="33.02" x2="36.195" y2="33.9725" width="1.016" layer="16"/>
-<wire x1="36.195" y1="33.9725" x2="36.195" y2="36.195" width="1.016" layer="16"/>
 <wire x1="32.0675" y1="35.8775" x2="35.8775" y2="35.8775" width="1.27" layer="16"/>
 <wire x1="35.8775" y1="35.8775" x2="36.195" y2="36.195" width="1.27" layer="16"/>
@@
 <wire x1="32.0675" y1="31.115" x2="32.0675" y2="35.8775" width="1.27" layer="16"/>
 <wire x1="32.0675" y1="31.115" x2="24.6075" y2="31.115" width="1.27" layer="16"/>
+<wire x1="38.735" y1="32.7025" x2="37.1475" y2="31.115" width="1.016" layer="16"/>
+<wire x1="37.1475" y1="31.115" x2="34.925" y2="31.115" width="1.016" layer="16"/>
 </signal>
 <signal name="V15+">
@@
 <contactref element="R8" pad="2"/>
 <wire x1="29.3675" y1="40.64" x2="30.7975" y2="40.64" width="1.016" layer="16"/>
-<wire x1="30.7975" y1="40.64" x2="32.0675" y2="41.275" width="1.016" layer="16"/>
-<wire x1="32.0675" y1="41.275" x2="43.815" y2="41.275" width="1.016" layer="16"/>
-<wire x1="43.815" y1="41.275" x2="44.7675" y2="40.9575" width="1.016" layer="16"/>
+<wire x1="30.7975" y1="40.64" x2="31.90875" y2="41.11625" width="1.016" layer="16"/>
+<wire x1="31.90875" y1="41.11625" x2="43.815" y2="41.11625" width="1.016" layer="16"/>
+<wire x1="43.815" y1="41.11625" x2="44.7675" y2="40.9575" width="1.016" layer="16"/>
 <contactref element="DA1" pad="11"/>
 <wire x1="19.05" y1="21.2725" x2="20.6375" y2="21.2725" width="1.016" layer="16"/>

Commit message: 7
Parts:
- added SJ4: (no value), jumper:SJ
- C7: device resistor:C025-025X050 -> resistor:C050-025X075
- GND, OUT, V+, V-: value (none) -> CON_2PA
- IN: device DSS0:CON_PWR_2PIN4MM -> woofer:CON_PWRI_2PIN4MM
- moved R8 5.30 mm to (23.5, 26.5), turned to 90 degrees
- moved VD2 1.14 mm to (9.53, 8.57)
- moved C8 0.81 mm to (3.97, 15.1)
- moved SJ2 0.81 mm to (24.3, 23.0)
- moved C7 0.79 mm to (8.10, 14.9), turned to 90 degrees
- moved R3 0.79 mm to (9.84, 21.9), turned to 270 degrees
- moved R5 0.64 mm to (20.0, 6.03)
- moved SJ1 0.35 mm to (16.0, 17.1)
- moved DA1 0.32 mm to (16.8, 21.0)
- moved SJ3 0.32 mm to (18.1, 26.0)
Connections:
- new net N$8: DA1.11, SJ4.1
- net VC+: now also SJ4.2; no longer DA1.11
Routing:
- net N$8: track 0.00 -> 3.87 mm
- net CO: track 11.2 -> 13.9 mm
- net VC+: track 48.6 -> 51.2 mm, vias 0 -> 1
- net C-: track 27.6 -> 29.8 mm
- net L-OUT: track 158.7 -> 158.1 mm
- net VC-: track 43.5 -> 43.6 mm, vias 0 -> 1

Commit message: 8
Parts:
- moved C5 0.71 mm to (14.6, 31.1)
- moved SJ3 0.64 mm to (18.1, 25.4)
- moved SJ4 0.64 mm to (17.3, 22.4)
- moved DA1 0.63 mm to (16.8, 20.3)
- moved R3 0.63 mm to (9.84, 21.3)
- moved SJ1 0.63 mm to (16.0, 16.5)
- moved R8 0.32 mm to (23.5, 26.2)
- moved SJ2 0.32 mm to (24.3, 22.7)
Routing:
- net GND: track 386.6 -> 387.5 mm
- net C+: track 16.3 -> 17.1 mm
- net N$16: track 12.9 -> 12.2 mm
- net NL: track 77.5 -> 76.9 mm

Commit message: 9
Parts:
- C10: device resistor:C025-025X050 -> resistor:C050-025X075
- C3: device resistor:C025-030X050 -> resistor:C050-025X075
- C4: device resistor:C025-025X050 -> C:C_11X3.5
- R4, R5: device resistor:0207/10 -> resistor:M1206
- moved R4 5.02 mm to (25.7, 9.84), flipped to the bottom, turned to 0 degrees
- moved C4 4.55 mm to (27.0, 7.62), turned to 270 degrees
- moved R5 2.42 mm to (21.0, 3.81), flipped to the bottom, turned to 90 degrees
- moved R14 1.27 mm to (42.2, 7.62)
- moved VD9 0.64 mm to (53.0, 40.0)
- moved C10 0.32 mm to (34.6, 7.62)
- moved R7 0.32 mm to (16.5, 2.54)
- moved VD6 0.32 mm to (50.5, 5.08)
Connections:
- removed net N$23: C4.2, R4.2
- new net N$7: C4.1, R4.1
- net C-: now also R4.2; no longer C4.1
- net L-OUT: now also C4.2; no longer R4.1
Routing:
- net L-OUT: track 158.1 -> 152.2 mm
- net N$7: track 0.00 -> 3.37 mm
- net V-: track 136.5 -> 139.8 mm
- net N$23: track 1.90 -> 0.00 mm
- net N$13: track 5.71 -> 4.63 mm
- net N$50: track 13.4 -> 14.2 mm
- net N$10: track 5.86 -> 6.45 mm

Commit message: 10
Parts:
- moved R4 3.51 mm to (25.4, 6.35)
- moved VT1 1.27 mm to (26.4, 15.2)
- moved C4 1.27 mm to (27.0, 6.35)
Routing:
- net V-: track 139.8 -> 138.1 mm
- net GND: track 387.3 -> 388.6 mm
- net N$50: track 14.2 -> 13.0 mm
- net N$7: track 3.37 -> 4.62 mm
- net CO: track 14.0 -> 15.0 mm
Changed lines of the file:
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@@
 <layer number="24" name="bOrigins" color="15" fill="1" visible="yes" active="yes"/>
 <layer number="25" name="tNames" color="7" fill="1" visible="yes" active="yes"/>
-<layer number="26" name="bNames" color="7" fill="1" visible="yes" active="yes"/>
-<layer number="27" name="tValues" color="7" fill="1" visible="no" active="yes"/>
+<layer number="26" name="bNames" color="7" fill="1" visible="no" active="yes"/>
+<layer number="27" name="tValues" color="7" fill="1" visible="yes" active="yes"/>
 <layer number="28" name="bValues" color="7" fill="1" visible="no" active="yes"/>
 <layer number="29" name="tStop" color="7" fill="3" visible="no" active="yes"/>
@@
 <dimension x1="144.145" y1="45.72" x2="144.145" y2="-1.5875" x3="149.225" y3="22.06625" layer="47" dtype="vertical"/>
 <dimension x1="-0.635" y1="-4.1275" x2="141.605" y2="-3.4925" x3="70.485" y3="-9.8425" layer="47" dtype="horizontal"/>
-<dimension x1="154.6225" y1="22.225" x2="167.64" y2="19.05" x3="-27.305" y3="20.6375" layer="47" dtype="vertical"/>
-<dimension x1="55.40375" y1="48.73625" x2="45.4025" y2="46.83125" x3="50.403125" y3="-26.67" layer="47" dtype="horizontal"/>
+<dimension x1="154.6225" y1="22.225" x2="153.035" y2="18.415" x3="-27.305" y3="20.32" layer="47" dtype="vertical"/>
+<dimension x1="-6.19125" y1="50.64125" x2="-3.175" y2="50.00625" x3="-4.683125" y3="-26.67" layer="47" dtype="horizontal"/>
 </plain>
 <attributes>
@@
 </autorouter>
 <elements>
-<element name="VT1" library="transistor" package="TO92-CBE" value="2N5401" x="26.3525" y="16.51" smashed="yes" rot="R180">
-<attribute name="NAME" x="26.51125" y="21.3995" size="1.27" layer="25" ratio="10" rot="R180"/>
-<attribute name="VALUE" x="23.1775" y="18.288" size="1.27" layer="27" ratio="10"/>
+<element name="VT1" library="transistor" package="TO92-CBE" value="2N5401" x="26.3525" y="15.24" smashed="yes" rot="R180">
+<attribute name="NAME" x="26.51125" y="20.1295" size="1.27" layer="25" ratio="10" rot="R180"/>
+<attribute name="VALUE" x="23.1775" y="17.3355" size="1.27" layer="27" ratio="10"/>
 </element>
 <element name="C10" library="resistor" package="C050-025X075" value="750" x="34.6075" y="7.62" smashed="yes">
-<attribute name="NAME" x="32.131" y="8.636" size="1.27" layer="25" ratio="10" rot="R180"/>
-<attribute name="VALUE" x="31.8135" y="7.239" size="1.27" layer="27" ratio="10" rot="R180"/>
+<attribute name="NAME" x="34.3535" y="2.921" size="1.27" layer="25" ratio="10" rot="R180"/>
+<attribute name="VALUE" x="35.814" y="1.651" size="1.27" layer="27" ratio="10"/>
 </element>
 <element name="R10" library="resistor" package="RTRIM3296W" value="10k" x="29.5275" y="22.86" smashed="yes" rot="R180">
@@
 <attribute name="VALUE" x="19.7231" y="3.4925" size="1.27" layer="28" ratio="10" rot="MR0"/>
 </element>
-<element name="C4" library="C" package="C_11X3.5" value="100" x="26.9875" y="7.62" smashed="yes" rot="R270">
-<attribute name="NAME" x="26.289" y="6.4135" size="1.27" layer="25" ratio="10" rot="R270"/>
-<attribute name="VALUE" x="26.0985" y="10.8585" size="1.27" layer="27" ratio="10" rot="R270"/>
-</element>
-<element name="R4" library="resistor" package="M1206" value="6k8" x="25.7175" y="9.8425" smashed="yes" rot="MR0">
-<attribute name="NAME" x="28.1305" y="7.239" size="1.27" layer="26" ratio="10" rot="MR0"/>
-<attribute name="VALUE" x="28.2956" y="5.715" size="1.27" layer="28" ratio="10" rot="MR0"/>
+<element name="C4" library="C" package="C_11X3.5" value="100" x="26.9875" y="6.35" smashed="yes" rot="R270">
+<attribute name="NAME" x="25.875" y="6.155" size="1.27" layer="25"/>
+<attribute name="VALUE" x="28.3675" y="5.7525" size="1.27" layer="27" rot="R180"/>
+</element>
+<element name="R4" library="resistor" package="M1206" value="6k8" x="25.4" y="6.35" smashed="yes" rot="MR0">
+<attribute name="NAME" x="27.813" y="2.159" size="1.27" layer="26" ratio="10" rot="MR0"/>
+<attribute name="VALUE" x="27.9781" y="2.2225" size="1.27" layer="28" ratio="10" rot="MR0"/>
 </element>
 <element name="R3" library="resistor" package="M0805" value="1k" x="9.8425" y="21.2725" smashed="yes" rot="MR270">
@@
 </element>
 <element name="DA2" library="IC" package="DIL8" value="IR2153D" x="39.37" y="8.89" smashed="yes" rot="R270">
-<attribute name="NAME" x="37.719" y="9.5885" size="1.27" layer="25" ratio="10"/>
-<attribute name="VALUE" x="37.43325" y="6.985" size="1.27" layer="27" ratio="10"/>
+<attribute name="NAME" x="37.719" y="16.5735" size="1.27" layer="25" ratio="10"/>
+<attribute name="VALUE" x="38.38575" y="6.35" size="1.27" layer="27" ratio="10"/>
 </element>
 <element name="R17" library="resistor" package="M1206" value="10k" x="55.08625" y="27.94" smashed="yes" rot="MR90">
@@
 </element>
 <element name="DA1" library="IC" package="DIL_A(14)" value="K554CA3" x="16.8275" y="20.32" smashed="yes">
-<attribute name="NAME" x="14.4145" y="27.051" size="1.27" layer="25" ratio="10"/>
+<attribute name="NAME" x="15.0495" y="27.051" size="1.27" layer="25" ratio="10"/>
 <attribute name="VALUE" x="17.145" y="20.701" size="1.27" layer="27" ratio="10" rot="R270"/>
 </element>
@@
 <wire x1="44.9725" y1="31.115" x2="44.9725" y2="30.685" width="1.27" layer="16"/>
 <wire x1="44.9725" y1="30.685" x2="40.9575" y2="26.67" width="1.27" layer="16"/>
-<wire x1="30.48" y1="2.2225" x2="27.6225" y2="5.08" width="1.27" layer="16"/>
-<wire x1="27.6225" y1="5.08" x2="25.0825" y2="5.08" width="1.27" layer="16"/>
-<wire x1="25.0825" y1="5.08" x2="24.13" y2="4.1275" width="1.27" layer="16"/>
-<wire x1="24.13" y1="4.1275" x2="24.13" y2="2.54" width="1.27" layer="16"/>
+<wire x1="30.48" y1="2.2225" x2="28.575" y2="4.1275" width="1.27" layer="16"/>
+<wire x1="28.575" y1="4.1275" x2="25.7175" y2="4.1275" width="1.27" layer="16"/>
+<wire x1="25.7175" y1="4.1275" x2="24.13" y2="2.54" width="1.27" layer="16"/>
 </signal>
 <signal name="GND">
@@
 <wire x1="53.81625" y1="36.5125" x2="54.7225" y2="38.2125" width="1.016" layer="16"/>
 <wire x1="54.7225" y1="38.2125" x2="54.7225" y2="40.005" width="1.016" layer="16"/>
-<wire x1="26.3525" y1="16.51" x2="26.3525" y2="18.57375" width="1.016" layer="16"/>
+<wire x1="26.3525" y1="15.24" x2="26.3525" y2="18.57375" width="1.016" layer="16"/>
 <wire x1="26.3525" y1="18.57375" x2="27.14625" y2="19.3675" width="1.016" layer="16"/>
 <wire x1="32.0675" y1="43.4975" x2="32.0675" y2="43.815" width="1.27" layer="16"/>
@@
 <wire x1="30.1625" y1="12.065" x2="30.1625" y2="13.0175" width="1.016" layer="16"/>
 <wire x1="30.1625" y1="13.0175" x2="28.8925" y2="14.2875" width="1.016" layer="16"/>
-<wire x1="28.8925" y1="14.2875" x2="28.8925" y2="16.51" width="1.016" layer="16"/>
+<wire x1="28.8925" y1="14.2875" x2="28.8925" y2="15.24" width="1.016" layer="16"/>
 <wire x1="31.4325" y1="4.7625" x2="29.21" y2="6.985" width="1.016" layer="16"/>
 <wire x1="29.21" y1="6.985" x2="29.21" y2="9.8425" width="1.016" layer="16"/>
@@
 <wire x1="21.59" y1="0" x2="20.955" y2="0.635" width="0.8128" layer="16"/>
 <wire x1="20.955" y1="0.635" x2="20.955" y2="2.41" width="0.8128" layer="16"/>
-<wire x1="26.9875" y1="2.0825" x2="26.9875" y2="0" width="0.8128" layer="16"/>
+<wire x1="26.9875" y1="1.8125" x2="26.9875" y2="0" width="0.8128" layer="16"/>
 </signal>
 <signal name="N$28">
@@
 <contactref element="DA1" pad="(3)"/>
 <wire x1="9.8425" y1="20.3225" x2="13.0175" y2="20.32" width="1.016" layer="16"/>
-<wire x1="18.415" y1="10.795" x2="23.365" y2="10.795" width="0.8128" layer="16"/>
+<wire x1="18.415" y1="10.795" x2="23.1775" y2="10.795" width="0.8128" layer="16"/>
 <wire x1="18.415" y1="10.795" x2="17.30375" y2="11.90625" width="0.8128" layer="16"/>
 <wire x1="17.30375" y1="11.90625" x2="17.30375" y2="14.12875" width="0.8128" layer="16"/>
 <wire x1="17.30375" y1="14.12875" x2="17.93875" y2="14.76375" width="0.8128" layer="16"/>
 <contactref element="R4" pad="2"/>
-<wire x1="23.365" y1="10.795" x2="24.3175" y2="9.8425" width="0.8128" layer="16"/>
-<wire x1="20.955" y1="5.21" x2="22.0375" y2="5.21" width="0.8128" layer="16"/>
-<wire x1="22.0375" y1="5.21" x2="24.3175" y2="7.49" width="0.8128" layer="16"/>
-<wire x1="24.3175" y1="7.49" x2="24.3175" y2="9.8425" width="0.8128" layer="16"/>
+<wire x1="23.1775" y1="10.795" x2="24.4475" y2="9.525" width="0.8128" layer="16"/>
+<wire x1="24.4475" y1="9.525" x2="24.4475" y2="8.255" width="0.8128" layer="16"/>
+<wire x1="24.4475" y1="8.255" x2="24" y2="7.49" width="0.8128" layer="16"/>
+<wire x1="24" y1="7.49" x2="24" y2="6.35" width="0.8128" layer="16"/>
+<wire x1="20.955" y1="5.21" x2="22.86" y2="5.21" width="0.8128" layer="16"/>
+<wire x1="22.86" y1="5.21" x2="24" y2="6.35" width="0.8128" layer="16"/>
 </signal>
 <signal name="CO">
@@
 <contactref element="VT1" pad="E"/>
 <contactref element="DA1" pad="9"/>
-<wire x1="20.6375" y1="15.24" x2="23.8125" y2="16.51" width="1.016" layer="16"/>
+<wire x1="20.6375" y1="15.24" x2="23.8125" y2="15.24" width="1.016" layer="16"/>
 <wire x1="25.05075" y1="22.70125" x2="25.05075" y2="24.79675" width="0.8128" layer="16"/>
 <wire x1="25.05075" y1="24.79675" x2="24.60375" y2="25.24375" width="0.8128" layer="16"/>
 <wire x1="24.60375" y1="25.24375" x2="23.495" y2="25.24375" width="0.8128" layer="16"/>
-<wire x1="23.8125" y1="16.51" x2="23.8125" y2="19.05" width="1.016" layer="16"/>
+<wire x1="23.8125" y1="15.24" x2="23.8125" y2="19.05" width="1.016" layer="16"/>
 <wire x1="23.8125" y1="19.05" x2="25.05075" y2="20.28825" width="1.016" layer="16"/>
 <wire x1="25.05075" y1="20.28825" x2="25.05075" y2="22.70125" width="1.016" layer="16"/>
@@
 <contactref element="R4" pad="1"/>
 <contactref element="C4" pad="1"/>
-<wire x1="27.1175" y1="9.8425" x2="27.1175" y2="13.0275" width="1.016" layer="16"/>
-<wire x1="27.1175" y1="13.0275" x2="26.9875" y2="13.1575" width="1.016" layer="16"/>
+<wire x1="26.8" y1="6.35" x2="26.8" y2="10.7" width="0.8128" layer="16"/>
+<wire x1="26.8" y1="10.7" x2="26.9875" y2="10.8875" width="0.8128" layer="16"/>
 </signal>
 </signals>

Commit message: rel 1
Parts:
- GND, OUT, V+, V-: value CON_2PA -> (none)
- VT2: device transistor:TO220V -> m_transistor:TO220FV
- VT3, VT4: device woofer:TO126V -> m_transistor:TO126V
- moved SJ2 6.75 mm to (18.1, 25.4), turned to 0 degrees
- moved SJ3 6.75 mm to (24.3, 22.7), turned to 180 degrees
- moved SJ1 6.01 mm to (17.3, 22.4)
- moved SJ4 6.01 mm to (16.0, 16.5)
- moved C5 0.32 mm to (14.6, 30.8)
- turned R10 to 0 degrees
Connections:
- net CO: now also SJ3.2; no longer SJ2.2
- net N$1: now also R10.3; no longer R10.1
- net N$35: now also SJ3.1; no longer SJ2.1
- net N$37: now also SJ4.2; no longer SJ1.2
- net N$40: now also SJ2.1; no longer SJ3.1
- net N$6: now also R10.1; no longer R10.3
- net N$8: now also SJ1.1; no longer SJ4.1
- net VC+: now also SJ1.2, SJ2.2; no longer SJ3.2, SJ4.2
- net VC-: now also SJ4.1; no longer SJ1.1
Routing:
- net NL: track 76.9 -> 78.4 mm
- net N$1: track 13.4 -> 14.1 mm
- net N$12: track 7.33 -> 7.95 mm
