File: WooferAmpIR2153.brd (EAGLE design)
At the start: 142.2 x 47.3 mm, 71 parts

Commit message: rel 2
Parts:
- C2: device resistor:C025-030X050 -> resistor:C050-025X075
- IN: value (none) -> CON_2PB
- R12: device resistor:0204/7 -> resistor:0207/10
- R4: device resistor:M1206 -> resistor:M0805
- moved R4 6.38 mm to (24.8, 12.7)
- moved R5 5.17 mm to (24.4, 7.62)
- moved VT1 0.63 mm to (26.4, 15.9)
- moved R12 0.63 mm to (32.1, 39.1)
- moved C2 0.32 mm to (7.30, 29.8)
- moved C4 0.32 mm to (27.0, 6.03)
Routing:
- net L-OUT: track 151.9 -> 156.8 mm
- net C-: track 30.5 -> 26.5 mm
- net GND: track 388.5 -> 385.1 mm
- net N$2: track 23.8 -> 22.4 mm
- net N$7: track 4.62 -> 5.29 mm, vias 0 -> 1
- net N$50: track 13.0 -> 13.6 mm
- net CO: track 15.0 -> 14.4 mm

Commit message: fix2
Parts:
- C11: device resistor:C025-025X050 -> resistor:C050-025X075
- moved C11 0.95 mm to (35.9, 23.8)
Routing:
- net V-: track 138.4 -> 134.6 mm
- net GND: track 385.1 -> 386.6 mm
- net L-OUT: track 156.8 -> 157.6 mm
Changed lines of the file:
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@@
 <layer number="26" name="bNames" color="7" fill="1" visible="yes" active="yes"/>
 <layer number="27" name="tValues" color="7" fill="1" visible="no" active="yes"/>
-<layer number="28" name="bValues" color="7" fill="1" visible="no" active="yes"/>
+<layer number="28" name="bValues" color="7" fill="1" visible="yes" active="yes"/>
 <layer number="29" name="tStop" color="7" fill="3" visible="no" active="yes"/>
 <layer number="30" name="bStop" color="7" fill="6" visible="no" active="yes"/>
@@
 <attribute name="VALUE" x="26.0731" y="17.78" size="1.27" layer="28" ratio="10" rot="MR0"/>
 </element>
-<element name="C11" library="resistor" package="C025-025X050" value="100n" x="34.925" y="23.8125" smashed="yes">
-<attribute name="NAME" x="32.639" y="26.924" size="1.27" layer="25" ratio="10"/>
-<attribute name="VALUE" x="32.639" y="25.146" size="1.27" layer="27" ratio="10"/>
+<element name="C11" library="resistor" package="C050-025X075" value="100n" x="35.8775" y="23.8125" smashed="yes">
+<attribute name="NAME" x="33.5915" y="26.924" size="1.27" layer="25" ratio="10"/>
+<attribute name="VALUE" x="33.5915" y="25.146" size="1.27" layer="27" ratio="10"/>
 </element>
 <element name="C12" library="resistor" package="E2,5-6" value="47m" x="39.6875" y="26.67" smashed="yes">
@@
 </element>
 <element name="R13" library="resistor" package="M1206" value="39" x="41.43375" y="21.43125" smashed="yes" rot="MR90">
-<attribute name="NAME" x="40.98925" y="23.90775" size="1.27" layer="26" ratio="10" rot="MR0"/>
-<attribute name="VALUE" x="39.88435" y="22.38375" size="1.27" layer="28" ratio="10" rot="MR0"/>
+<attribute name="NAME" x="42.57675" y="24.22525" size="1.27" layer="26" ratio="10" rot="MR0"/>
+<attribute name="VALUE" x="37.34435" y="24.28875" size="1.27" layer="28" ratio="10" rot="MR0"/>
 </element>
 <element name="R14" library="resistor" package="M1206" value="39" x="42.2275" y="7.62" smashed="yes" rot="MR180">
@@
 <wire x1="61.357346875" y1="5.794846875" x2="61.039846875" y2="5.878465625" width="1.016" layer="16"/>
 <contactref element="VD4" pad="A"/>
-<wire x1="36.195" y1="23.8125" x2="39.37" y2="24.4475" width="0.8128" layer="16"/>
+<wire x1="38.4175" y1="23.8125" x2="39.37" y2="24.4475" width="0.8128" layer="16"/>
 <wire x1="39.37" y1="24.4475" x2="40.9575" y2="26.67" width="0.8128" layer="16"/>
 <wire x1="38.4175" y1="11.1125" x2="38.4175" y2="19.685" width="0.8128" layer="16"/>
@@
 <wire x1="39.0525" y1="20.32" x2="39.0525" y2="22.5425" width="0.8128" layer="16"/>
 <wire x1="39.0525" y1="22.5425" x2="38.4175" y2="23.1775" width="0.8128" layer="16"/>
-<wire x1="38.4175" y1="23.1775" x2="36.195" y2="23.8125" width="0.8128" layer="16"/>
+<wire x1="38.4175" y1="23.1775" x2="38.4175" y2="23.8125" width="0.8128" layer="16"/>
 <wire x1="43.815" y1="32.7025" x2="44.9725" y2="31.115" width="1.27" layer="16"/>
 <wire x1="44.9725" y1="31.115" x2="44.9725" y2="30.685" width="1.27" layer="16"/>
@@
 <wire x1="88.9" y1="22.86" x2="82.55" y2="22.86" width="2.1844" layer="16"/>
 <wire x1="111.03" y1="34.29" x2="97.79" y2="34.29" width="2.1844" layer="16"/>
-<wire x1="137.16" y1="24.13" x2="137.16" y2="37.7825" width="2.1844" layer="16"/>
-<wire x1="137.16" y1="24.13" x2="137.795" y2="11.39" width="2.1844" layer="16"/>
+<wire x1="139.16" y1="24.13" x2="139.16" y2="37.7825" width="2.1844" layer="16"/>
+<wire x1="139.16" y1="24.13" x2="137.795" y2="11.39" width="2.1844" layer="16"/>
 <wire x1="137.795" y1="11.39" x2="139.3425" y2="8.255" width="2.1844" layer="16"/>
-<wire x1="137.16" y1="37.7825" x2="135.5725" y2="35.56" width="2.1844" layer="16"/>
+<wire x1="139.16" y1="37.7825" x2="135.5725" y2="35.56" width="2.1844" layer="16"/>
 <wire x1="135.5725" y1="35.56" x2="130.81" y2="35.56" width="2.1844" layer="16"/>
 <wire x1="129.2225" y1="43.18" x2="114.935" y2="43.18" width="2.1844" layer="16"/>
@@
 <wire x1="111.03" y1="8.89" x2="109.4425" y2="8.89" width="2.1844" layer="16"/>
 <wire x1="118.4675" y1="8.255" x2="115.57" y2="10.16" width="2.1844" layer="16"/>
-<wire x1="121.285" y1="37.7825" x2="121.285" y2="24.13" width="2.1844" layer="16"/>
-<wire x1="121.285" y1="24.13" x2="121.285" y2="14.2875" width="2.1844" layer="16"/>
+<wire x1="119.285" y1="37.7825" x2="119.285" y2="24.13" width="2.1844" layer="16"/>
 <wire x1="121.285" y1="14.2875" x2="115.57" y2="10.16" width="2.1844" layer="16"/>
 <wire x1="99.3775" y1="8.89" x2="109.4425" y2="8.89" width="1.27" layer="16"/>
@@
 <wire x1="115.03" y1="3.4925" x2="115.03" y2="10.16" width="2.1844" layer="16"/>
 <wire x1="115.03" y1="10.16" x2="115.57" y2="10.16" width="2.1844" layer="16"/>
-<polygon width="0.254" layer="16" thermals="no">
-<vertex x="124.1425" y="38.1"/>
-<vertex x="120.3325" y="38.1"/>
-<vertex x="120.3325" y="12.3825"/>
-<vertex x="124.1425" y="15.24"/>
-</polygon>
 <polygon width="0.254" layer="16" thermals="no">
 <vertex x="111.125" y="2.54"/>
@@
 <wire x1="59.3725" y1="0" x2="60.325" y2="0" width="1.016" layer="16"/>
 <wire x1="60.325" y1="0" x2="60.6425" y2="0.3175" width="1.016" layer="16"/>
+<polygon width="0.254" layer="16" thermals="no">
+<vertex x="118.4275" y="40.9575"/>
+<vertex x="118.4275" y="20.0025"/>
+<vertex x="120.3325" y="18.0975"/>
+<vertex x="120.3325" y="15.875"/>
+<vertex x="116.5225" y="12.065"/>
+<vertex x="116.5225" y="9.525"/>
+<vertex x="121.92" y="9.525"/>
+<vertex x="125.73" y="13.335"/>
+<vertex x="125.73" y="40.64"/>
+<vertex x="125.4125" y="40.9575"/>
+</polygon>
+<wire x1="121.285" y1="14.2875" x2="121.285" y2="22.13" width="2.1844" layer="16"/>
+<wire x1="121.285" y1="22.13" x2="119.285" y2="24.13" width="2.1844" layer="16"/>
 </signal>
 <signal name="N$28">
@@
 <contactref element="C12" pad="+"/>
 <wire x1="35.56" y1="17.78" x2="35.2425" y2="21.2725" width="1.016" layer="16"/>
-<wire x1="35.2425" y1="21.2725" x2="33.655" y2="23.8125" width="1.016" layer="16"/>
-<wire x1="33.655" y1="23.8125" x2="34.29" y2="25.0825" width="1.27" layer="16"/>
+<wire x1="35.2425" y1="21.2725" x2="33.3375" y2="23.8125" width="1.016" layer="16"/>
+<wire x1="33.3375" y1="23.8125" x2="34.29" y2="25.0825" width="1.27" layer="16"/>
 <wire x1="34.29" y1="25.0825" x2="35.8775" y2="26.67" width="1.27" layer="16"/>
 <wire x1="35.8775" y1="26.67" x2="38.4175" y2="26.67" width="1.27" layer="16"/>

Commit message: hm10
Parts:
- C1: value 10m -> (none)
- C10: device resistor:C050-025X075 -> resistor:C075-032X103
- moved R14 1.91 mm to (44.1, 7.62)
- moved C10 1.31 mm to (35.9, 7.30)
Routing:
- net V-: track 134.6 -> 136.9 mm
- net N$13: track 4.63 -> 3.20 mm
- net N$15: track 9.49 -> 8.94 mm
Changed lines of the file:
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@@
 <attribute name="VALUE" x="23.1775" y="17.9705" size="1.27" layer="27" ratio="10"/>
 </element>
-<element name="C10" library="resistor" package="C050-025X075" value="750" x="34.6075" y="7.62" smashed="yes">
-<attribute name="NAME" x="34.3535" y="2.921" size="1.27" layer="25" ratio="10" rot="R180"/>
-<attribute name="VALUE" x="35.814" y="1.651" size="1.27" layer="27" ratio="10"/>
+<element name="C10" library="resistor" package="C075-032X103" value="750" x="35.8775" y="7.3025" smashed="yes">
+<attribute name="NAME" x="35.6235" y="2.6035" size="1.27" layer="25" ratio="10" rot="R180"/>
+<attribute name="VALUE" x="37.084" y="1.3335" size="1.27" layer="27" ratio="10"/>
 </element>
 <element name="R10" library="resistor" package="RTRIM3296W" value="10k" x="29.5275" y="22.86" smashed="yes">
@@
 <attribute name="VALUE" x="37.34435" y="24.28875" size="1.27" layer="28" ratio="10" rot="MR0"/>
 </element>
-<element name="R14" library="resistor" package="M1206" value="39" x="42.2275" y="7.62" smashed="yes" rot="MR180">
-<attribute name="NAME" x="37.75075" y="12.446" size="1.27" layer="26" ratio="10" rot="MR180"/>
-<attribute name="VALUE" x="38.3794" y="10.795" size="1.27" layer="28" ratio="10" rot="MR180"/>
+<element name="R14" library="resistor" package="M1206" value="39" x="44.1325" y="7.62" smashed="yes" rot="MR180">
+<attribute name="NAME" x="38.70325" y="12.446" size="1.27" layer="26" ratio="10" rot="MR180"/>
+<attribute name="VALUE" x="39.0144" y="10.795" size="1.27" layer="28" ratio="10" rot="MR180"/>
 </element>
 <element name="VT4" library="m_transistor" package="TO126V" value="BD138" x="49.8475" y="9.525" smashed="yes" rot="R180">
@@
 <attribute name="VALUE" x="43.2435" y="34.036" size="1.27" layer="27" ratio="10"/>
 </element>
-<element name="C1" library="resistor" package="E2,5-6" value="10m" x="3.175" y="29.845" smashed="yes" rot="R90">
+<element name="C1" library="resistor" package="E2,5-6" value="" x="3.175" y="29.845" smashed="yes" rot="R90">
 <attribute name="NAME" x="-0.1905" y="34.8615" size="1.27" layer="25" ratio="10"/>
 <attribute name="VALUE" x="-0.1905" y="32.5755" size="1.27" layer="27" ratio="10"/>
@@
 <wire x1="41.5925" y1="4.7625" x2="41.5925" y2="3.175" width="1.016" layer="16"/>
 <wire x1="41.5925" y1="3.175" x2="41.91" y2="2.2225" width="1.016" layer="16"/>
-<wire x1="37.1475" y1="7.62" x2="37.1475" y2="2.2225" width="1.016" layer="16"/>
-<wire x1="37.1475" y1="7.62" x2="35.56" y2="10.16" width="1.016" layer="16"/>
+<wire x1="39.6875" y1="7.3025" x2="37.1475" y2="2.2225" width="1.016" layer="16"/>
+<wire x1="39.6875" y1="7.3025" x2="35.56" y2="10.16" width="1.016" layer="16"/>
 <wire x1="35.56" y1="10.16" x2="37.465" y2="10.16" width="1.016" layer="16"/>
 <wire x1="37.465" y1="10.16" x2="38.4175" y2="11.1125" width="1.016" layer="16"/>
@@
 <wire x1="54.7225" y1="40.005" x2="54.7225" y2="42.6575" width="1.016" layer="16"/>
 <wire x1="54.7225" y1="42.6575" x2="55.245" y2="43.815" width="1.016" layer="16"/>
-<wire x1="66.3575" y1="25.2095" x2="66.3575" y2="19.2405" width="2.54" layer="16"/>
+<wire x1="66.3575" y1="25.2095" x2="66.3575" y2="19.2405" width="3" layer="16"/>
 <wire x1="79.375" y1="30.7975" x2="82.55" y2="27.6225" width="2.1844" layer="16"/>
 <wire x1="82.55" y1="27.6225" x2="82.55" y2="22.86" width="2.1844" layer="16"/>
 <wire x1="82.55" y1="22.86" x2="82.55" y2="13.335" width="2.1844" layer="16"/>
 <wire x1="82.55" y1="13.335" x2="79.375" y2="13.335" width="2.7" layer="16"/>
-<wire x1="66.3575" y1="25.2095" x2="70.358" y2="29.21" width="2.54" layer="16"/>
+<wire x1="66.3575" y1="25.2095" x2="70.358" y2="29.21" width="3" layer="16"/>
 <wire x1="70.358" y1="29.21" x2="77.47" y2="29.21" width="2.1844" layer="16"/>
 <wire x1="77.47" y1="29.21" x2="79.0575" y2="30.7975" width="2.1844" layer="16"/>
@@
 </polygon>
 <polygon width="0.254" layer="16" thermals="no">
-<vertex x="81.28" y="34.925"/>
-<vertex x="74.6125" y="34.925"/>
-<vertex x="69.5325" y="29.845"/>
-<vertex x="69.5325" y="27.94"/>
-<vertex x="81.28" y="27.94"/>
-</polygon>
-<polygon width="0.254" layer="16" thermals="no">
-<vertex x="127.9525" y="44.45"/>
-<vertex x="127.9525" y="10.16"/>
+<vertex x="128.905" y="44.7675"/>
+<vertex x="128.905" y="10.4775"/>
 <vertex x="118.745" y="4.445"/>
 <vertex x="118.745" y="2.54"/>
@@
 <wire x1="30.1625" y1="37.7825" x2="24.4475" y2="34.925" width="1.016" layer="16"/>
 <wire x1="24.4475" y1="34.925" x2="23.1775" y2="34.925" width="1.016" layer="16"/>
+<polygon width="0.254" layer="16" thermals="no">
+<vertex x="110.1725" y="43.4975"/>
+<vertex x="110.1725" y="34.29"/>
+<vertex x="116.205" y="34.29"/>
+<vertex x="116.205" y="43.4975"/>
+</polygon>
+<polygon width="0.254" layer="16" thermals="no">
+<vertex x="66.675" y="18.0975"/>
+<vertex x="70.1675" y="21.59"/>
+<vertex x="70.1675" y="24.765"/>
+<vertex x="72.39" y="26.9875"/>
+<vertex x="80.645" y="26.9875"/>
+<vertex x="80.645" y="34.925"/>
+<vertex x="74.295" y="34.925"/>
+<vertex x="66.3575" y="27.305"/>
+<vertex x="66.3575" y="18.0975"/>
+</polygon>
 </signal>
 <signal name="N$4">
@@
 <wire x1="33.655" y1="12.7" x2="35.56" y2="12.7" width="1.016" layer="16"/>
 <wire x1="32.7025" y1="12.065" x2="32.0675" y2="9.2075" width="1.016" layer="16"/>
-<wire x1="32.0675" y1="9.2075" x2="32.0675" y2="7.62" width="1.016" layer="16"/>
+<wire x1="32.0675" y1="9.2075" x2="32.0675" y2="7.3025" width="1.016" layer="16"/>
 <wire x1="32.7025" y1="12.065" x2="32.7025" y2="13.335" width="1.016" layer="16"/>
 <wire x1="32.7025" y1="13.335" x2="31.115" y2="14.9225" width="1.016" layer="16"/>
@@
 <contactref element="VD6" pad="A"/>
 <contactref element="R14" pad="2"/>
-<wire x1="45.4025" y1="5.08" x2="43.6275" y2="7.62" width="1.016" layer="16"/>
+<wire x1="45.4025" y1="5.08" x2="45.5325" y2="7.62" width="1.016" layer="16"/>
 <wire x1="47.244" y1="10.795" x2="47.244" y2="7.239" width="1.016" layer="16"/>
 <wire x1="47.244" y1="7.239" x2="45.4025" y2="5.08" width="1.016" layer="16"/>
@@
 <vertex x="116.5225" y="9.525"/>
 <vertex x="121.92" y="9.525"/>
-<vertex x="125.73" y="13.335"/>
-<vertex x="125.73" y="40.64"/>
+<vertex x="126.365" y="13.97"/>
+<vertex x="126.365" y="40.64"/>
 <vertex x="125.4125" y="40.9575"/>
 </polygon>
@@
 <contactref element="DA2" pad="5"/>
 <contactref element="R14" pad="1"/>
-<wire x1="40.8275" y1="7.62" x2="40.8275" y2="9.7125" width="1.016" layer="16"/>
-<wire x1="40.8275" y1="9.7125" x2="41.275" y2="10.16" width="1.016" layer="16"/>
-<wire x1="41.275" y1="10.16" x2="43.18" y2="10.16" width="1.016" layer="16"/>
+<wire x1="42.7325" y1="7.62" x2="42.7325" y2="9.395" width="1.016" layer="16"/>
+<wire x1="42.7325" y1="9.395" x2="42.545" y2="10.16" width="1.016" layer="16"/>
+<wire x1="42.545" y1="10.16" x2="43.18" y2="10.16" width="1.016" layer="16"/>
 </signal>
 <signal name="NL">
@@
 <wire x1="74.93" y1="20.32" x2="70.1675" y2="15.5575" width="1.778" layer="16"/>
 <wire x1="70.1675" y1="15.5575" x2="62.23" y2="15.5575" width="1.778" layer="16"/>
-<wire x1="62.23" y1="15.5575" x2="62.23" y2="17.4625" width="1.778" layer="16"/>
-<wire x1="62.23" y1="17.4625" x2="60.6425" y2="19.05" width="1.778" layer="16"/>
+<wire x1="62.23" y1="15.5575" x2="62.23" y2="17.4625" width="2.54" layer="16"/>
+<wire x1="62.23" y1="17.4625" x2="60.6425" y2="19.05" width="2.54" layer="16"/>
 <wire x1="62.23" y1="15.5575" x2="62.23" y2="11.1125" width="1.778" layer="16"/>
 <wire x1="62.23" y1="11.1125" x2="58.42" y2="11.1125" width="1.778" layer="16"/>
@@
 <wire x1="49.8475" y1="20.6375" x2="49.824078125" y2="20.37985625" width="1.778" layer="16"/>
 <wire x1="49.824078125" y1="20.37985625" x2="49.53" y2="17.145" width="1.778" layer="16"/>
-<wire x1="60.6425" y1="25.7175" x2="60.6425" y2="19.05" width="1.9304" layer="16"/>
+<wire x1="60.6425" y1="25.7175" x2="60.6425" y2="19.05" width="2.54" layer="16"/>
 <wire x1="55.08625" y1="26.54" x2="56.385" y2="26.54" width="1.016" layer="16"/>
 <wire x1="56.385" y1="26.54" x2="58.42" y2="27.94" width="1.016" layer="16"/>
-<wire x1="58.42" y1="27.94" x2="60.6425" y2="25.7175" width="1.9304" layer="16"/>
+<wire x1="58.42" y1="27.94" x2="60.6425" y2="25.7175" width="2.1844" layer="16"/>
 <wire x1="55.5625" y1="19.05" x2="54.23264375" y2="20.37985625" width="1.9304" layer="16"/>
 <wire x1="54.23264375" y1="20.37985625" x2="49.824078125" y2="20.37985625" width="1.9304" layer="16"/>
+<polygon width="0.254" layer="16" thermals="no">
+<vertex x="58.42" y="27.94"/>
+<vertex x="58.7375" y="16.51"/>
+<vertex x="63.5" y="14.605"/>
+<vertex x="63.5" y="27.94"/>
+</polygon>
 </signal>
 <signal name="N$2">
