File: WooferAmpIR2153.brd (EAGLE design)
At the start: 142.2 x 47.3 mm, 71 parts

Commit message: rel3
Parts:
- moved R9 3.27 mm to (34.9, 7.62)
- moved C10 2.62 mm to (35.2, 4.76)
- moved R14 0.32 mm to (44.5, 7.62)
Routing:
- net N$50: track 13.6 -> 9.11 mm
- net N$4: track 13.0 -> 16.5 mm
- net V-: track 136.9 -> 138.7 mm
Changed lines of the file:
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@@
 <attribute name="VALUE" x="23.1775" y="17.9705" size="1.27" layer="27" ratio="10"/>
 </element>
-<element name="C10" library="resistor" package="C075-032X103" value="750" x="35.8775" y="7.3025" smashed="yes">
-<attribute name="NAME" x="35.6235" y="2.6035" size="1.27" layer="25" ratio="10" rot="R180"/>
-<attribute name="VALUE" x="37.084" y="1.3335" size="1.27" layer="27" ratio="10"/>
+<element name="C10" library="resistor" package="C075-032X103" value="750" x="35.2425" y="4.7625" smashed="yes">
+<attribute name="NAME" x="34.9885" y="0.0635" size="1.27" layer="25" ratio="10" rot="R180"/>
+<attribute name="VALUE" x="36.449" y="-1.2065" size="1.27" layer="27" ratio="10"/>
 </element>
 <element name="R10" library="resistor" package="RTRIM3296W" value="10k" x="29.5275" y="22.86" smashed="yes">
@@
 <attribute name="VALUE" x="37.34435" y="24.28875" size="1.27" layer="28" ratio="10" rot="MR0"/>
 </element>
-<element name="R14" library="resistor" package="M1206" value="39" x="44.1325" y="7.62" smashed="yes" rot="MR180">
-<attribute name="NAME" x="38.70325" y="12.446" size="1.27" layer="26" ratio="10" rot="MR180"/>
-<attribute name="VALUE" x="39.0144" y="10.795" size="1.27" layer="28" ratio="10" rot="MR180"/>
+<element name="R14" library="resistor" package="M1206" value="39" x="44.45" y="7.62" smashed="yes" rot="MR180">
+<attribute name="NAME" x="38.38575" y="12.446" size="1.27" layer="26" ratio="10" rot="MR180"/>
+<attribute name="VALUE" x="38.6969" y="10.795" size="1.27" layer="28" ratio="10" rot="MR180"/>
 </element>
 <element name="VT4" library="m_transistor" package="TO126V" value="BD138" x="49.8475" y="9.525" smashed="yes" rot="R180">
@@
 <attribute name="VALUE" x="51.55565" y="19.20875" size="1.27" layer="28" ratio="10" rot="MR180"/>
 </element>
-<element name="R9" library="resistor" package="0207/10" value="3k3" x="36.5125" y="4.7625" smashed="yes">
-<attribute name="NAME" x="33.782" y="4.064" size="1.27" layer="25" ratio="10"/>
-<attribute name="VALUE" x="36.7919" y="4.1275" size="1.27" layer="27" ratio="10"/>
+<element name="R9" library="resistor" package="0207/10" value="3k3" x="34.925" y="7.62" smashed="yes">
+<attribute name="NAME" x="32.1945" y="6.9215" size="1.27" layer="25" ratio="10"/>
+<attribute name="VALUE" x="35.2044" y="6.985" size="1.27" layer="27" ratio="10"/>
 </element>
 <element name="R6" library="resistor" package="P0613/15" value="2k2 1w" x="52.3875" y="40.9575" smashed="yes">
@@
 <contactref element="C11" pad="2"/>
 <contactref element="C13" pad="2"/>
-<wire x1="30.48" y1="2.2225" x2="37.1475" y2="2.2225" width="1.778" layer="16"/>
-<wire x1="37.1475" y1="2.2225" x2="41.91" y2="2.2225" width="1.778" layer="16"/>
+<wire x1="30.1625" y1="2.2225" x2="39.37" y2="2.2225" width="1.778" layer="16"/>
+<wire x1="39.37" y1="2.2225" x2="41.91" y2="2.2225" width="1.778" layer="16"/>
 <wire x1="41.91" y1="2.2225" x2="49.8475" y2="2.2225" width="1.778" layer="16"/>
 <wire x1="49.8475" y1="2.2225" x2="58.1025" y2="2.2225" width="1.778" layer="16"/>
-<wire x1="41.5925" y1="4.7625" x2="41.5925" y2="3.175" width="1.016" layer="16"/>
-<wire x1="41.5925" y1="3.175" x2="41.91" y2="2.2225" width="1.016" layer="16"/>
-<wire x1="39.6875" y1="7.3025" x2="37.1475" y2="2.2225" width="1.016" layer="16"/>
-<wire x1="39.6875" y1="7.3025" x2="35.56" y2="10.16" width="1.016" layer="16"/>
+<wire x1="39.0525" y1="4.7625" x2="35.56" y2="10.16" width="1.016" layer="16"/>
 <wire x1="35.56" y1="10.16" x2="37.465" y2="10.16" width="1.016" layer="16"/>
 <wire x1="37.465" y1="10.16" x2="38.4175" y2="11.1125" width="1.016" layer="16"/>
@@
 <wire x1="44.9725" y1="31.115" x2="44.9725" y2="30.685" width="1.27" layer="16"/>
 <wire x1="44.9725" y1="30.685" x2="40.9575" y2="26.67" width="1.27" layer="16"/>
-<wire x1="30.48" y1="2.2225" x2="28.575" y2="4.1275" width="1.27" layer="16"/>
-<wire x1="28.575" y1="4.1275" x2="25.7175" y2="4.1275" width="1.27" layer="16"/>
+<wire x1="30.1625" y1="2.2225" x2="28.2575" y2="4.1275" width="1.27" layer="16"/>
+<wire x1="28.2575" y1="4.1275" x2="25.7175" y2="4.1275" width="1.27" layer="16"/>
 <wire x1="25.7175" y1="4.1275" x2="24.13" y2="2.54" width="1.27" layer="16"/>
 <wire x1="58.42" y1="8.5725" x2="56.0675" y2="8.5725" width="1.016" layer="16"/>
 <wire x1="56.0675" y1="8.5725" x2="55.08625" y2="9.55375" width="1.016" layer="16"/>
+<wire x1="39.0525" y1="4.7625" x2="39.37" y2="2.2225" width="1.27" layer="16"/>
+<wire x1="40.005" y1="7.62" x2="41.91" y2="5.08" width="1.016" layer="16"/>
+<wire x1="41.91" y1="5.08" x2="41.91" y2="2.2225" width="1.016" layer="16"/>
 </signal>
 <signal name="GND">
@@
 <wire x1="32.7025" y1="12.065" x2="33.655" y2="12.7" width="1.016" layer="16"/>
 <wire x1="33.655" y1="12.7" x2="35.56" y2="12.7" width="1.016" layer="16"/>
-<wire x1="32.7025" y1="12.065" x2="32.0675" y2="9.2075" width="1.016" layer="16"/>
-<wire x1="32.0675" y1="9.2075" x2="32.0675" y2="7.3025" width="1.016" layer="16"/>
 <wire x1="32.7025" y1="12.065" x2="32.7025" y2="13.335" width="1.016" layer="16"/>
 <wire x1="32.7025" y1="13.335" x2="31.115" y2="14.9225" width="1.016" layer="16"/>
 <wire x1="31.115" y1="14.9225" x2="31.115" y2="16.5125" width="1.016" layer="16"/>
+<wire x1="32.7025" y1="12.065" x2="32.0675" y2="11.43" width="1.016" layer="16"/>
+<wire x1="32.0675" y1="11.43" x2="32.0675" y2="9.2075" width="1.016" layer="16"/>
+<wire x1="32.0675" y1="9.2075" x2="32.7025" y2="8.5725" width="1.016" layer="16"/>
+<wire x1="32.7025" y1="8.5725" x2="32.7025" y2="6.0325" width="1.016" layer="16"/>
+<wire x1="32.7025" y1="6.0325" x2="31.4325" y2="4.7625" width="1.016" layer="16"/>
 </signal>
 <signal name="VB">
@@
 <contactref element="VD6" pad="A"/>
 <contactref element="R14" pad="2"/>
-<wire x1="45.4025" y1="5.08" x2="45.5325" y2="7.62" width="1.016" layer="16"/>
+<wire x1="45.4025" y1="5.08" x2="45.85" y2="7.62" width="1.016" layer="16"/>
 <wire x1="47.244" y1="10.795" x2="47.244" y2="7.239" width="1.016" layer="16"/>
 <wire x1="47.244" y1="7.239" x2="45.4025" y2="5.08" width="1.016" layer="16"/>
@@
 <contactref element="R9" pad="1"/>
 <contactref element="C9" pad="-"/>
-<wire x1="31.4325" y1="4.7625" x2="31.115" y2="4.7625" width="1.016" layer="16"/>
 <wire x1="30.1625" y1="12.065" x2="30.1625" y2="12.3825" width="1.016" layer="16"/>
 <wire x1="30.1625" y1="12.065" x2="30.1625" y2="13.0175" width="1.016" layer="16"/>
 <wire x1="30.1625" y1="13.0175" x2="28.8925" y2="14.2875" width="1.016" layer="16"/>
 <wire x1="28.8925" y1="14.2875" x2="28.8925" y2="15.875" width="1.016" layer="16"/>
-<wire x1="31.4325" y1="4.7625" x2="29.21" y2="6.985" width="1.016" layer="16"/>
-<wire x1="29.21" y1="6.985" x2="29.21" y2="9.8425" width="1.016" layer="16"/>
-<wire x1="29.21" y1="9.8425" x2="30.1625" y2="10.795" width="1.016" layer="16"/>
-<wire x1="30.1625" y1="10.795" x2="30.1625" y2="12.065" width="1.016" layer="16"/>
+<wire x1="29.845" y1="7.62" x2="30.1625" y2="12.065" width="1.016" layer="16"/>
 </signal>
 <signal name="VC-">
@@
 <contactref element="DA2" pad="5"/>
 <contactref element="R14" pad="1"/>
-<wire x1="42.7325" y1="7.62" x2="42.7325" y2="9.395" width="1.016" layer="16"/>
+<wire x1="43.05" y1="7.62" x2="42.7325" y2="9.395" width="1.016" layer="16"/>
 <wire x1="42.7325" y1="9.395" x2="42.545" y2="10.16" width="1.016" layer="16"/>
 <wire x1="42.545" y1="10.16" x2="43.18" y2="10.16" width="1.016" layer="16"/>

Commit message: rel4
Parts:
- VT1: device transistor:TO92-CBE -> m_transistor:TO92
- moved VT1 1.27 mm to (26.4, 17.1), turned to 0 degrees
Connections:
- net CO: now also VT1.1; no longer VT1.E
- net GND: now also VT1.2; no longer VT1.B
- net N$50: now also VT1.3; no longer VT1.C
Changed lines of the file:
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@@
 </autorouter>
 <elements>
-<element name="VT1" library="transistor" package="TO92-CBE" value="2N5401" x="26.3525" y="15.875" smashed="yes" rot="R180">
-<attribute name="NAME" x="26.51125" y="20.7645" size="1.27" layer="25" ratio="10" rot="R180"/>
-<attribute name="VALUE" x="23.1775" y="17.9705" size="1.27" layer="27" ratio="10"/>
+<element name="VT1" library="m_transistor" package="TO92" value="2N5401" x="26.3525" y="17.145" smashed="yes">
+<attribute name="NAME" x="25.87625" y="20.5105" size="1.27" layer="25" ratio="10"/>
+<attribute name="VALUE" x="29.5275" y="15.0495" size="1.27" layer="27" ratio="10" rot="R180"/>
 </element>
 <element name="C10" library="resistor" package="C075-032X103" value="750" x="35.2425" y="4.7625" smashed="yes">
@@
 <element name="R11" library="resistor" package="M0805" value="750" x="31.115" y="17.4625" smashed="yes" rot="MR270">
 <attribute name="NAME" x="26.63825" y="18.95475" size="1.27" layer="26" ratio="10" rot="MR180"/>
-<attribute name="VALUE" x="26.0731" y="17.78" size="1.27" layer="28" ratio="10" rot="MR0"/>
+<attribute name="VALUE" x="26.0731" y="18.0975" size="1.27" layer="28" ratio="10" rot="MR0"/>
 </element>
 <element name="C11" library="resistor" package="C050-025X075" value="100n" x="35.8775" y="23.8125" smashed="yes">
@@
 <contactref element="C17" pad="2"/>
 <contactref element="VT2" pad="2"/>
-<contactref element="VT1" pad="B"/>
+<contactref element="VT1" pad="2"/>
 <contactref element="R12" pad="1"/>
 <contactref element="C3" pad="1"/>
@@
 </signal>
 <signal name="N$50">
-<contactref element="VT1" pad="C"/>
+<contactref element="VT1" pad="3"/>
 <contactref element="R9" pad="1"/>
 <contactref element="C9" pad="-"/>
@@
 <contactref element="R8" pad="1"/>
 <contactref element="SJ3" pad="2"/>
-<contactref element="VT1" pad="E"/>
+<contactref element="VT1" pad="1"/>
 <contactref element="DA1" pad="9"/>
 <wire x1="20.6375" y1="15.24" x2="23.8125" y2="15.875" width="1.016" layer="16"/>
