File: WooferAmpIR2153.sch (EAGLE design)
At the start: 70 parts

Commit message: .
Parts:
- removed C14B: (no value), resistor:C-EU075-032X103
Connections:
- net NL: no longer C14B.2
- net VB: no longer C14B.1
Changed lines of the file:
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@@
 <?xml version="1.0" encoding="utf-8"?>
 <!DOCTYPE eagle SYSTEM "eagle.dtd">
-<eagle version="6.3">
+<eagle version="6.4">
 <drawing>
 <settings>
@@
 <grid distance="100" unitdist="mil" unit="mil" style="lines" multiple="1" display="yes" altdistance="0.01" altunitdist="inch" altunit="inch"/>
 <layers>
-<layer number="1" name="Top" color="4" fill="1" visible="yes" active="no"/>
-<layer number="2" name="Route2" color="1" fill="3" visible="yes" active="no"/>
-<layer number="3" name="Route3" color="4" fill="3" visible="yes" active="no"/>
-<layer number="4" name="Route4" color="1" fill="4" visible="yes" active="no"/>
-<layer number="5" name="Route5" color="4" fill="4" visible="yes" active="no"/>
-<layer number="6" name="Route6" color="1" fill="8" visible="yes" active="no"/>
-<layer number="7" name="Route7" color="4" fill="8" visible="yes" active="no"/>
-<layer number="8" name="Route8" color="1" fill="2" visible="yes" active="no"/>
-<layer number="9" name="Route9" color="4" fill="2" visible="yes" active="no"/>
-<layer number="10" name="Route10" color="1" fill="7" visible="yes" active="no"/>
-<layer number="11" name="Route11" color="4" fill="7" visible="yes" active="no"/>
-<layer number="12" name="Route12" color="1" fill="5" visible="yes" active="no"/>
-<layer number="13" name="Route13" color="4" fill="5" visible="yes" active="no"/>
-<layer number="14" name="Route14" color="1" fill="6" visible="yes" active="no"/>
-<layer number="15" name="Route15" color="4" fill="6" visible="yes" active="no"/>
-<layer number="16" name="Bottom" color="1" fill="1" visible="yes" active="no"/>
-<layer number="17" name="Pads" color="2" fill="1" visible="yes" active="no"/>
-<layer number="18" name="Vias" color="2" fill="1" visible="yes" active="no"/>
-<layer number="19" name="Unrouted" color="6" fill="1" visible="yes" active="no"/>
-<layer number="20" name="Dimension" color="15" fill="1" visible="yes" active="no"/>
-<layer number="21" name="tPlace" color="7" fill="1" visible="yes" active="no"/>
-<layer number="22" name="bPlace" color="7" fill="1" visible="yes" active="no"/>
-<layer number="23" name="tOrigins" color="15" fill="1" visible="yes" active="no"/>
-<layer number="24" name="bOrigins" color="15" fill="1" visible="yes" active="no"/>
-<layer number="25" name="tNames" color="7" fill="1" visible="yes" active="no"/>
-<layer number="26" name="bNames" color="7" fill="1" visible="yes" active="no"/>
-<layer number="27" name="tValues" color="7" fill="1" visible="yes" active="no"/>
-<layer number="28" name="bValues" color="7" fill="1" visible="yes" active="no"/>
+<layer number="1" name="Top" color="4" fill="1" visible="no" active="no"/>
+<layer number="2" name="Route2" color="1" fill="3" visible="no" active="no"/>
+<layer number="3" name="Route3" color="4" fill="3" visible="no" active="no"/>
+<layer number="4" name="Route4" color="1" fill="4" visible="no" active="no"/>
+<layer number="5" name="Route5" color="4" fill="4" visible="no" active="no"/>
+<layer number="6" name="Route6" color="1" fill="8" visible="no" active="no"/>
+<layer number="7" name="Route7" color="4" fill="8" visible="no" active="no"/>
+<layer number="8" name="Route8" color="1" fill="2" visible="no" active="no"/>
+<layer number="9" name="Route9" color="4" fill="2" visible="no" active="no"/>
+<layer number="10" name="Route10" color="1" fill="7" visible="no" active="no"/>
+<layer number="11" name="Route11" color="4" fill="7" visible="no" active="no"/>
+<layer number="12" name="Route12" color="1" fill="5" visible="no" active="no"/>
+<layer number="13" name="Route13" color="4" fill="5" visible="no" active="no"/>
+<layer number="14" name="Route14" color="1" fill="6" visible="no" active="no"/>
+<layer number="15" name="Route15" color="4" fill="6" visible="no" active="no"/>
+<layer number="16" name="Bottom" color="1" fill="1" visible="no" active="no"/>
+<layer number="17" name="Pads" color="2" fill="1" visible="no" active="no"/>
+<layer number="18" name="Vias" color="2" fill="1" visible="no" active="no"/>
+<layer number="19" name="Unrouted" color="6" fill="1" visible="no" active="no"/>
+<layer number="20" name="Dimension" color="15" fill="1" visible="no" active="no"/>
+<layer number="21" name="tPlace" color="7" fill="1" visible="no" active="no"/>
+<layer number="22" name="bPlace" color="7" fill="1" visible="no" active="no"/>
+<layer number="23" name="tOrigins" color="15" fill="1" visible="no" active="no"/>
+<layer number="24" name="bOrigins" color="15" fill="1" visible="no" active="no"/>
+<layer number="25" name="tNames" color="7" fill="1" visible="no" active="no"/>
+<layer number="26" name="bNames" color="7" fill="1" visible="no" active="no"/>
+<layer number="27" name="tValues" color="7" fill="1" visible="no" active="no"/>
+<layer number="28" name="bValues" color="7" fill="1" visible="no" active="no"/>
 <layer number="29" name="tStop" color="7" fill="3" visible="no" active="no"/>
 <layer number="30" name="bStop" color="7" fill="6" visible="no" active="no"/>
@@
 <layer number="35" name="tGlue" color="7" fill="4" visible="no" active="no"/>
 <layer number="36" name="bGlue" color="7" fill="5" visible="no" active="no"/>
-<layer number="37" name="tTest" color="7" fill="1" visible="yes" active="no"/>
-<layer number="38" name="bTest" color="7" fill="1" visible="yes" active="no"/>
+<layer number="37" name="tTest" color="7" fill="1" visible="no" active="no"/>
+<layer number="38" name="bTest" color="7" fill="1" visible="no" active="no"/>
 <layer number="39" name="tKeepout" color="4" fill="11" visible="no" active="no"/>
 <layer number="40" name="bKeepout" color="1" fill="11" visible="no" active="no"/>
@@
 <layer number="44" name="Drills" color="7" fill="1" visible="no" active="no"/>
 <layer number="45" name="Holes" color="7" fill="1" visible="no" active="no"/>
-<layer number="46" name="Milling" color="3" fill="1" visible="yes" active="no"/>
-<layer number="47" name="Measures" color="7" fill="1" visible="yes" active="no"/>
-<layer number="48" name="Document" color="7" fill="1" visible="yes" active="no"/>
-<layer number="49" name="Reference" color="7" fill="1" visible="yes" active="no"/>
-<layer number="50" name="dxf" color="7" fill="1" visible="yes" active="no"/>
-<layer number="51" name="tDocu" color="7" fill="1" visible="yes" active="no"/>
-<layer number="52" name="bDocu" color="7" fill="1" visible="yes" active="no"/>
-<layer number="53" name="tGND_GNDA" color="7" fill="1" visible="yes" active="no"/>
-<layer number="54" name="bGND_GNDA" color="7" fill="1" visible="yes" active="no"/>
-<layer number="56" name="wert" color="7" fill="1" visible="yes" active="no"/>
-<layer number="57" name="tCAD" color="7" fill="1" visible="yes" active="no"/>
+<layer number="46" name="Milling" color="3" fill="1" visible="no" active="no"/>
+<layer number="47" name="Measures" color="7" fill="1" visible="no" active="no"/>
+<layer number="48" name="Document" color="7" fill="1" visible="no" active="no"/>
+<layer number="49" name="Reference" color="7" fill="1" visible="no" active="no"/>
+<layer number="50" name="dxf" color="7" fill="1" visible="no" active="no"/>
+<layer number="51" name="tDocu" color="7" fill="1" visible="no" active="no"/>
+<layer number="52" name="bDocu" color="7" fill="1" visible="no" active="no"/>
+<layer number="53" name="tGND_GNDA" color="7" fill="1" visible="no" active="no"/>
+<layer number="54" name="bGND_GNDA" color="7" fill="1" visible="no" active="no"/>
+<layer number="56" name="wert" color="7" fill="1" visible="no" active="no"/>
+<layer number="57" name="tCAD" color="7" fill="1" visible="no" active="no"/>
 <layer number="90" name="Modules" color="13" fill="1" visible="yes" active="yes"/>
 <layer number="91" name="Nets" color="2" fill="1" visible="yes" active="yes"/>
@@
 <part name="OUT" library="woofer" deviceset="CON_2P" device="" value=""/>
 <part name="GND" library="woofer" deviceset="CON_2P" device="" value=""/>
-<part name="C14B" library="resistor" deviceset="C-EU" device="075-032X103"/>
 </parts>
 <sheets>
@@
 <instance part="OUT" gate="G$1" x="248.92" y="134.62" rot="R180"/>
 <instance part="GND" gate="G$1" x="248.92" y="149.86" rot="R180"/>
-<instance part="C14B" gate="G$1" x="132.08" y="157.48" smashed="yes" rot="R90">
-<attribute name="NAME" x="128.524" y="160.401" size="1.778" layer="95"/>
-<attribute name="VALUE" x="133.604" y="160.401" size="1.778" layer="96"/>
-</instance>
 </instances>
 <busses>
@@
 <wire x1="106.68" y1="149.86" x2="116.84" y2="149.86" width="0.1524" layer="91"/>
 <junction x="116.84" y="149.86"/>
-<pinref part="C14B" gate="G$1" pin="1"/>
 <wire x1="129.54" y1="157.48" x2="124.46" y2="157.48" width="0.1524" layer="91"/>
 <wire x1="124.46" y1="157.48" x2="124.46" y2="149.86" width="0.1524" layer="91"/>
@@
 <wire x1="157.48" y1="127" x2="157.48" y2="124.46" width="0.1524" layer="91"/>
 <pinref part="U$4" gate="G$1" pin="1"/>
-<pinref part="C14B" gate="G$1" pin="2"/>
 <wire x1="137.16" y1="157.48" x2="142.24" y2="157.48" width="0.1524" layer="91"/>
 <wire x1="142.24" y1="157.48" x2="142.24" y2="149.86" width="0.1524" layer="91"/>

Commit message: 2
Parts:
- added VD10: Д814В, DSS0:ZDD814
Changed lines of the file:
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@@
 <part name="OUT" library="woofer" deviceset="CON_2P" device="" value=""/>
 <part name="GND" library="woofer" deviceset="CON_2P" device="" value=""/>
+<part name="VD10" library="DSS0" deviceset="ZD" device="D814" value="Д814В"/>
 </parts>
 <sheets>
@@
 <instance part="OUT" gate="G$1" x="248.92" y="134.62" rot="R180"/>
 <instance part="GND" gate="G$1" x="248.92" y="149.86" rot="R180"/>
+<instance part="VD10" gate="G$1" x="73.66" y="48.26" smashed="yes" rot="R180">
+<attribute name="NAME" x="84.582" y="52.705" size="1.778" layer="95"/>
+<attribute name="VALUE" x="84.582" y="49.911" size="1.778" layer="96"/>
+</instance>
 </instances>
 <busses>
@@
 <pinref part="C14" gate="G$1" pin="+"/>
 <pinref part="DA2" gate="G$1" pin="VB"/>
-<wire x1="129.54" y1="149.86" x2="124.46" y2="149.86" width="0.1524" layer="91"/>
-<wire x1="124.46" y1="149.86" x2="116.84" y2="149.86" width="0.1524" layer="91"/>
+<wire x1="129.54" y1="149.86" x2="116.84" y2="149.86" width="0.1524" layer="91"/>
 <wire x1="116.84" y1="149.86" x2="116.84" y2="132.08" width="0.1524" layer="91"/>
 <wire x1="106.68" y1="147.32" x2="106.68" y2="149.86" width="0.1524" layer="91"/>
 <wire x1="106.68" y1="149.86" x2="116.84" y2="149.86" width="0.1524" layer="91"/>
 <junction x="116.84" y="149.86"/>
-<wire x1="129.54" y1="157.48" x2="124.46" y2="157.48" width="0.1524" layer="91"/>
-<wire x1="124.46" y1="157.48" x2="124.46" y2="149.86" width="0.1524" layer="91"/>
-<junction x="124.46" y="149.86"/>
 </segment>
 </net>
@@
 <pinref part="DA2" gate="G$1" pin="VS"/>
 <pinref part="C14" gate="G$1" pin="-"/>
-<wire x1="137.16" y1="149.86" x2="142.24" y2="149.86" width="0.1524" layer="91"/>
-<wire x1="142.24" y1="149.86" x2="147.32" y2="149.86" width="0.1524" layer="91"/>
+<wire x1="137.16" y1="149.86" x2="147.32" y2="149.86" width="0.1524" layer="91"/>
 <wire x1="147.32" y1="149.86" x2="147.32" y2="127" width="0.1524" layer="91"/>
 <wire x1="147.32" y1="127" x2="144.78" y2="127" width="0.1524" layer="91"/>
@@
 <wire x1="157.48" y1="127" x2="157.48" y2="124.46" width="0.1524" layer="91"/>
 <pinref part="U$4" gate="G$1" pin="1"/>
-<wire x1="137.16" y1="157.48" x2="142.24" y2="157.48" width="0.1524" layer="91"/>
-<wire x1="142.24" y1="157.48" x2="142.24" y2="149.86" width="0.1524" layer="91"/>
-<junction x="142.24" y="149.86"/>
-</segment>
-</net>
+</segment>
+</net>

Commit message: h1
Parts:
- added U$1: L-D30, woofer:L-D30
- R12: device resistor:R-EU_0207/10 -> resistor:R-EU_0204/7
- R3, R8: device resistor:R-EU_0207/10 -> resistor:R-EU_M0805
Connections:
- net N$21 renamed L-OUT
- net GND: now also U$1G$2.1, U$1G$3.1, U$1G$5.1, U$1G$6.1
- net N$2: now also VD10.C; no longer VD4.C
- net V-: now also VD10.A; no longer VD4.A
Other:
- moved on the sheet: VD10

Commit message: r3
Parts:
- R12: device resistor:R-EU_0204/7 -> resistor:R-EU_0207/5V
Changed lines of the file:
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@@
 <?xml version="1.0" encoding="utf-8"?>
 <!DOCTYPE eagle SYSTEM "eagle.dtd">
-<eagle version="6.3">
+<eagle version="6.4">
 <drawing>
 <settings>
@@
 <part name="VT2" library="transistor" deviceset="*-NPN-" device="TO220V" value="13005"/>
 <part name="GND15" library="supply1" deviceset="GND" device=""/>
-<part name="R12" library="resistor" deviceset="R-EU_" device="0204/7" value="15k"/>
+<part name="R12" library="resistor" deviceset="R-EU_" device="0207/5V" value="15k"/>
 <part name="VD4" library="diode" deviceset="ZENER-DIODE" device="ZD-10" value="15v"/>
 <part name="C13" library="resistor" deviceset="C-EU" device="050-025X075" value="100n"/>

Commit message: h2
Parts:
- R12: device resistor:R-EU_0207/5V -> resistor:R-EU_0204/7
Connections:
- net N$10: now also R19.1; no longer C19.2
- net N$9: now also C19.2, R19.2; no longer C19.1, R19.1
- net NL: now also C19.1; no longer R19.2
Other:
- moved on the sheet: C19, R19
Changed lines of the file:
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@@
 <?xml version="1.0" encoding="utf-8"?>
 <!DOCTYPE eagle SYSTEM "eagle.dtd">
-<eagle version="6.4">
+<eagle version="6.3">
 <drawing>
 <settings>
@@
 <layer number="45" name="Holes" color="7" fill="1" visible="no" active="no"/>
 <layer number="46" name="Milling" color="3" fill="1" visible="yes" active="no"/>
-<layer number="47" name="Measures" color="7" fill="1" visible="yes" active="no"/>
+<layer number="47" name="Measures" color="13" fill="1" visible="yes" active="no"/>
 <layer number="48" name="Document" color="7" fill="1" visible="yes" active="no"/>
 <layer number="49" name="Reference" color="7" fill="1" visible="yes" active="no"/>
@@
 <part name="VT2" library="transistor" deviceset="*-NPN-" device="TO220V" value="13005"/>
 <part name="GND15" library="supply1" deviceset="GND" device=""/>
-<part name="R12" library="resistor" deviceset="R-EU_" device="0207/5V" value="15k"/>
+<part name="R12" library="resistor" deviceset="R-EU_" device="0204/7" value="15k"/>
 <part name="VD4" library="diode" deviceset="ZENER-DIODE" device="ZD-10" value="15v"/>
 <part name="C13" library="resistor" deviceset="C-EU" device="050-025X075" value="100n"/>
@@
 <attribute name="VALUE" x="141.097" y="154.4574" size="1.778" layer="96" rot="R180"/>
 </instance>
-<instance part="R19" gate="G$1" x="210.82" y="129.54" smashed="yes" rot="R90">
-<attribute name="NAME" x="209.55" y="128.0414" size="1.778" layer="95" rot="R180"/>
-<attribute name="VALUE" x="209.55" y="125.222" size="1.778" layer="96" rot="R180"/>
-</instance>
-<instance part="C19" gate="G$1" x="210.82" y="119.38" rot="MR0"/>
+<instance part="R19" gate="G$1" x="210.82" y="119.38" smashed="yes" rot="R90">
+<attribute name="NAME" x="209.55" y="117.8814" size="1.778" layer="95" rot="R180"/>
+<attribute name="VALUE" x="209.55" y="115.062" size="1.778" layer="96" rot="R180"/>
+</instance>
+<instance part="C19" gate="G$1" x="210.82" y="132.08" rot="MR0"/>
 <instance part="FRAME1" gate="G$1" x="0" y="0"/>
 <instance part="FRAME1" gate="G$2" x="175.26" y="0"/>
@@
 </segment>
 </net>
-<net name="N$9" class="0">
-<segment>
-<pinref part="R19" gate="G$1" pin="1"/>
-<pinref part="C19" gate="G$1" pin="1"/>
-<wire x1="210.82" y1="124.46" x2="210.82" y2="121.92" width="0.1524" layer="91"/>
-</segment>
-</net>
 <net name="N$10" class="0">
 <segment>
 <pinref part="VD9" gate="G$1" pin="C"/>
-<pinref part="C19" gate="G$1" pin="2"/>
 <wire x1="210.82" y1="109.22" x2="210.82" y2="111.76" width="0.1524" layer="91"/>
-<wire x1="210.82" y1="111.76" x2="210.82" y2="114.3" width="0.1524" layer="91"/>
 <wire x1="210.82" y1="111.76" x2="218.44" y2="111.76" width="0.1524" layer="91"/>
 <pinref part="HL1" gate="G$1" pin="A"/>
 <wire x1="218.44" y1="111.76" x2="218.44" y2="109.22" width="0.1524" layer="91"/>
+<pinref part="R19" gate="G$1" pin="1"/>
+<wire x1="210.82" y1="114.3" x2="210.82" y2="111.76" width="0.1524" layer="91"/>
 <junction x="210.82" y="111.76"/>
 </segment>
@@
 <wire x1="200.66" y1="121.92" x2="200.66" y2="124.46" width="0.1524" layer="91"/>
 <junction x="200.66" y="124.46"/>
-<pinref part="R19" gate="G$1" pin="2"/>
-<wire x1="210.82" y1="134.62" x2="210.82" y2="137.16" width="0.1524" layer="91"/>
 <wire x1="213.36" y1="137.16" x2="210.82" y2="137.16" width="0.1524" layer="91"/>
-<junction x="210.82" y="137.16"/>
 <wire x1="210.82" y1="137.16" x2="205.74" y2="137.16" width="0.1524" layer="91"/>
 <wire x1="205.74" y1="134.62" x2="205.74" y2="137.16" width="0.1524" layer="91"/>
@@
 <wire x1="157.48" y1="127" x2="157.48" y2="124.46" width="0.1524" layer="91"/>
 <pinref part="U$4" gate="G$1" pin="1"/>
+<pinref part="C19" gate="G$1" pin="1"/>
+<wire x1="210.82" y1="134.62" x2="210.82" y2="137.16" width="0.1524" layer="91"/>
+<junction x="210.82" y="137.16"/>
 </segment>
 </net>
@@
 </segment>
 </net>
+<net name="N$9" class="0">
+<segment>
+<pinref part="R19" gate="G$1" pin="2"/>
+<pinref part="C19" gate="G$1" pin="2"/>
+<wire x1="210.82" y1="124.46" x2="210.82" y2="127" width="0.1524" layer="91"/>
+</segment>
+</net>

Commit message: h5
Parts:
- removed VD10: Д814В, DSS0:ZDD814
- VD4: value 15v -> Д814Д; device diode:ZENER-DIODEZD-10 -> DSS0:ZDD814
- VD7, VD8, VD9: value 1N4148 -> LL4148
Connections:
- net N$2: now also VD4.C; no longer VD10.C
- net V-: now also VD4.A; no longer VD10.A
Changed lines of the file:
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@@
 <part name="C19" library="resistor" deviceset="C-EU" device="050-025X075" value="1n"/>
 <part name="FRAME1" library="frames" deviceset="DINA4_L" device=""/>
-<part name="VD9" library="diode" deviceset="DIODE-" device="SOD80C" value="1N4148"/>
+<part name="VD9" library="diode" deviceset="DIODE-" device="SOD80C" value="LL4148"/>
 <part name="HL1" library="led" deviceset="LED" device="3MM"/>
 <part name="R13" library="resistor" deviceset="R-EU_" device="M1206" value="39"/>
@@
 <part name="R17" library="resistor" deviceset="R-EU_" device="M1206" value="10k"/>
 <part name="R18" library="resistor" deviceset="R-EU_" device="M1206" value="10k"/>
-<part name="VD7" library="diode" deviceset="DIODE-" device="SOD80C" value="1N4148"/>
-<part name="VD8" library="diode" deviceset="DIODE-" device="SOD80C" value="1N4148"/>
+<part name="VD7" library="diode" deviceset="DIODE-" device="SOD80C" value="LL4148"/>
+<part name="VD8" library="diode" deviceset="DIODE-" device="SOD80C" value="LL4148"/>
 <part name="VT2" library="transistor" deviceset="*-NPN-" device="TO220V" value="13005"/>
 <part name="GND15" library="supply1" deviceset="GND" device=""/>
 <part name="R12" library="resistor" deviceset="R-EU_" device="0204/7" value="15k"/>
-<part name="VD4" library="diode" deviceset="ZENER-DIODE" device="ZD-10" value="15v"/>
 <part name="C13" library="resistor" deviceset="C-EU" device="050-025X075" value="100n"/>
 <part name="GND1" library="supply1" deviceset="GND" device=""/>
@@
 <part name="OUT" library="woofer" deviceset="CON_2P" device="" value=""/>
 <part name="GND" library="woofer" deviceset="CON_2P" device="" value=""/>
-<part name="VD10" library="DSS0" deviceset="ZD" device="D814" value="Д814В"/>
+<part name="VD4" library="DSS0" deviceset="ZD" device="D814" value="Д814Д"/>
 <part name="U$1" library="woofer" deviceset="L-D30" device=""/>
 <part name="GND9" library="supply1" deviceset="GND" device=""/>
@@
 <attribute name="VALUE" x="105.41" y="80.518" size="1.778" layer="96"/>
 </instance>
-<instance part="VD4" gate="G$1" x="121.92" y="83.82" smashed="yes" rot="R180">
-<attribute name="NAME" x="120.142" y="85.725" size="1.778" layer="95"/>
-<attribute name="VALUE" x="120.142" y="80.391" size="1.778" layer="96"/>
-</instance>
 <instance part="C13" gate="G$1" x="121.92" y="91.44" smashed="yes" rot="R90">
-<attribute name="NAME" x="118.364" y="94.361" size="1.778" layer="95"/>
+<attribute name="NAME" x="115.824" y="94.361" size="1.778" layer="95"/>
 <attribute name="VALUE" x="123.444" y="94.361" size="1.778" layer="96"/>
 </instance>
@@
 <instance part="OUT" gate="G$1" x="248.92" y="134.62" rot="R180"/>
 <instance part="GND" gate="G$1" x="248.92" y="149.86" rot="R180"/>
-<instance part="VD10" gate="G$1" x="121.92" y="76.2" smashed="yes" rot="R180">
-<attribute name="NAME" x="132.842" y="80.645" size="1.778" layer="95"/>
-<attribute name="VALUE" x="132.842" y="77.851" size="1.778" layer="96"/>
+<instance part="VD4" gate="G$1" x="121.92" y="83.82" smashed="yes" rot="R180">
+<attribute name="NAME" x="120.142" y="85.725" size="1.778" layer="95"/>
+<attribute name="VALUE" x="120.142" y="80.391" size="1.778" layer="96"/>
 </instance>
 <instance part="U$1" gate="G$1" x="165.1" y="27.94"/>
@@
 <pinref part="V-" gate="G$1" pin="1"/>
 <pinref part="V-" gate="G$1" pin="2"/>
-<pinref part="VD10" gate="G$1" pin="A"/>
-<wire x1="124.46" y1="76.2" x2="129.54" y2="76.2" width="0.1524" layer="91"/>
-<wire x1="129.54" y1="76.2" x2="129.54" y2="91.44" width="0.1524" layer="91"/>
+<pinref part="VD4" gate="G$1" pin="A"/>
+<wire x1="124.46" y1="83.82" x2="129.54" y2="83.82" width="0.1524" layer="91"/>
+<wire x1="129.54" y1="83.82" x2="129.54" y2="91.44" width="0.1524" layer="91"/>
 </segment>
 </net>
@@
 <wire x1="114.3" y1="83.82" x2="116.84" y2="83.82" width="0.1524" layer="91"/>
 <junction x="116.84" y="83.82"/>
-<pinref part="VD10" gate="G$1" pin="C"/>
-<wire x1="119.38" y1="76.2" x2="116.84" y2="76.2" width="0.1524" layer="91"/>
-<wire x1="116.84" y1="76.2" x2="116.84" y2="83.82" width="0.1524" layer="91"/>
-</segment>
-</net>
+<pinref part="VD4" gate="G$1" pin="C"/>
+<wire x1="119.38" y1="83.82" x2="116.84" y2="83.82" width="0.1524" layer="91"/>
+</segment>
+</net>

Commit message: h6
Parts:
- VT3, VT4: device transistor:-PNP-TO126V -> woofer:-PNP-TO126V
Changed lines of the file:
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@@
 <part name="R13" library="resistor" deviceset="R-EU_" device="M1206" value="39"/>
 <part name="R14" library="resistor" deviceset="R-EU_" device="M1206" value="39"/>
-<part name="VT4" library="transistor" deviceset="*-PNP-" device="TO126V" value="BD138"/>
-<part name="VT3" library="transistor" deviceset="*-PNP-" device="TO126V" value="BD138"/>
+<part name="VT4" library="woofer" deviceset="*-PNP-" device="TO126V" value="BD138"/>
+<part name="VT3" library="woofer" deviceset="*-PNP-" device="TO126V" value="BD138"/>
 <part name="VD5" library="diode" deviceset="DIODE-" device="DO204-10" value="SF16"/>
 <part name="VD6" library="diode" deviceset="DIODE-" device="DO204-10" value="SF16"/>

Commit message: 7
Parts:
- added SJ4: (no value), jumper:SJ
- C7: device resistor:C-EU025-025X050 -> resistor:C-EU050-025X075
- GND, OUT, V+, V-: value CON_2P -> CON_2PA; device woofer:CON_2P -> woofer:CON_2PA
- IN: value CON_2P -> CON_2PB; device DSS0:CON_2P -> woofer:CON_2PB
Connections:
- new net N$8: DA1A.V+, SJ4.1
- net VC+: now also SJ4.2; no longer DA1A.V+
Other:
- note added: "Для 8 установить SJ1 SJ2 S3 Для 16 удалить установить SJ4"
- note removed: "Для 8 установить SJ1 SJ2 S3 Для 16 удалить"
- moved on the sheet: C5, C6, R6, R8, VD1
