File: WooferAmpIR2153.sch (EAGLE design)
At the start: 71 parts

Commit message: 9
Parts:
- C10: device resistor:C-EU025-025X050 -> resistor:C-EU050-025X075
- C3: device resistor:C-EU025-030X050 -> resistor:C-EU050-025X075
- C4: device resistor:C-EU025-025X050 -> C:C11X3.5
- R4, R5: device resistor:R-EU_0207/10 -> resistor:R-EU_M1206
Connections:
- removed net N$23: C4.2, R4.2
- new net N$7: C4.1, R4.1
- net C-: now also R4.2; no longer C4.1
- net L-OUT: now also C4.2; no longer R4.1
Other:
- moved on the sheet: R4
Changed lines of the file:
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@@
 <parts>
 <part name="VT1" library="transistor" deviceset="*-PNP-" device="TO92-CBE" technology="BF493S" value="2N5401"/>
-<part name="C10" library="resistor" deviceset="C-EU" device="025-025X050" value="750"/>
+<part name="C10" library="resistor" deviceset="C-EU" device="050-025X075" value="750"/>
 <part name="R10" library="resistor" deviceset="R-TRIMM" device="3296W" value="10k"/>
 <part name="R11" library="resistor" deviceset="R-EU_" device="M0805" value="750"/>
@@
 <part name="R6" library="resistor" deviceset="R-EU_" device="0613/15" value="2k2 1w"/>
 <part name="R7" library="resistor" deviceset="R-EU_" device="0613/15" value="2k2 1w"/>
-<part name="R5" library="resistor" deviceset="R-EU_" device="0207/10" value="68k"/>
-<part name="C4" library="resistor" deviceset="C-EU" device="025-025X050" value="100"/>
-<part name="R4" library="resistor" deviceset="R-EU_" device="0207/10" value="6k8"/>
+<part name="R5" library="resistor" deviceset="R-EU_" device="M1206" value="68k"/>
+<part name="C4" library="C" deviceset="C" device="11X3.5" value="100"/>
+<part name="R4" library="resistor" deviceset="R-EU_" device="M1206" value="6k8"/>
 <part name="R3" library="resistor" deviceset="R-EU_" device="M0805" value="1k"/>
 <part name="R2" library="resistor" deviceset="R-EU_" device="0207/10" value="1k"/>
@@
 <part name="GND1" library="supply1" deviceset="GND" device=""/>
 <part name="C1" library="resistor" deviceset="CPOL-EU" device="E2.5-6" value="10m"/>
-<part name="C3" library="resistor" deviceset="C-EU" device="025-030X050" value="2n2"/>
+<part name="C3" library="resistor" deviceset="C-EU" device="050-025X075" value="2n2"/>
 <part name="GND16" library="supply1" deviceset="GND" device=""/>
 <part name="GND17" library="supply1" deviceset="GND" device=""/>
@@
 <attribute name="VALUE" x="44.45" y="105.918" size="1.778" layer="96"/>
 </instance>
-<instance part="C4" gate="G$1" x="35.56" y="111.76"/>
-<instance part="R4" gate="G$1" x="35.56" y="99.06" smashed="yes" rot="R90">
-<attribute name="NAME" x="34.29" y="107.7214" size="1.778" layer="95" rot="R180"/>
-<attribute name="VALUE" x="34.29" y="104.902" size="1.778" layer="96" rot="R180"/>
+<instance part="C4" gate="C$" x="35.56" y="99.06"/>
+<instance part="R4" gate="G$1" x="35.56" y="109.22" smashed="yes" rot="R90">
+<attribute name="NAME" x="34.29" y="117.8814" size="1.778" layer="95" rot="R180"/>
+<attribute name="VALUE" x="34.29" y="115.062" size="1.778" layer="96" rot="R180"/>
 </instance>
 <instance part="R3" gate="G$1" x="27.94" y="109.22" smashed="yes" rot="R90">
@@
 <wire x1="43.18" y1="71.12" x2="43.18" y2="91.44" width="0.1524" layer="91"/>
 <pinref part="R5" gate="G$1" pin="1"/>
-<pinref part="R4" gate="G$1" pin="1"/>
 <wire x1="43.18" y1="91.44" x2="43.18" y2="96.52" width="0.1524" layer="91"/>
-<wire x1="35.56" y1="93.98" x2="35.56" y2="91.44" width="0.1524" layer="91"/>
 <wire x1="35.56" y1="91.44" x2="43.18" y2="91.44" width="0.1524" layer="91"/>
 <junction x="43.18" y="91.44"/>
@@
 <junction x="238.76" y="134.62"/>
 <label x="231.14" y="137.16" size="1.778" layer="95"/>
-</segment>
-</net>
-<net name="N$23" class="0">
-<segment>
-<pinref part="R4" gate="G$1" pin="2"/>
-<pinref part="C4" gate="G$1" pin="2"/>
-<wire x1="35.56" y1="104.14" x2="35.56" y2="106.68" width="0.1524" layer="91"/>
+<pinref part="C4" gate="C$" pin="2"/>
+<wire x1="35.56" y1="91.44" x2="35.56" y2="93.98" width="0.1524" layer="91"/>
 </segment>
 </net>
@@
 <pinref part="R5" gate="G$1" pin="2"/>
 <wire x1="43.18" y1="106.68" x2="43.18" y2="116.84" width="0.1524" layer="91"/>
-<pinref part="C4" gate="G$1" pin="1"/>
-<wire x1="35.56" y1="114.3" x2="35.56" y2="116.84" width="0.1524" layer="91"/>
-<wire x1="35.56" y1="116.84" x2="43.18" y2="116.84" width="0.1524" layer="91"/>
 <pinref part="R3" gate="G$1" pin="2"/>
 <wire x1="27.94" y1="114.3" x2="27.94" y2="116.84" width="0.1524" layer="91"/>
 <wire x1="27.94" y1="116.84" x2="35.56" y2="116.84" width="0.1524" layer="91"/>
-<junction x="35.56" y="116.84"/>
 <pinref part="DA1" gate="A" pin="-IN"/>
+<wire x1="35.56" y1="116.84" x2="43.18" y2="116.84" width="0.1524" layer="91"/>
 <wire x1="48.26" y1="116.84" x2="43.18" y2="116.84" width="0.1524" layer="91"/>
 <junction x="43.18" y="116.84"/>
 <label x="45.72" y="116.84" size="1.778" layer="95"/>
+<pinref part="R4" gate="G$1" pin="2"/>
+<wire x1="35.56" y1="114.3" x2="35.56" y2="116.84" width="0.1524" layer="91"/>
+<junction x="35.56" y="116.84"/>
 </segment>
 <segment>
@@
 </segment>
 </net>
+<net name="N$7" class="0">
+<segment>
+<pinref part="R4" gate="G$1" pin="1"/>
+<pinref part="C4" gate="C$" pin="1"/>
+<wire x1="35.56" y1="104.14" x2="35.56" y2="101.6" width="0.1524" layer="91"/>
+</segment>
+</net>

Commit message: 10
Changed lines of the file:
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@@
 <plain>
 <text x="45.72" y="101.6" size="1.778" layer="91">33k</text>
-<text x="30.48" y="99.06" size="1.778" layer="91">3k3</text>
+<text x="30.48" y="106.68" size="1.778" layer="91">3k3</text>
 <text x="10.16" y="15.24" size="1.778" layer="91">Для  8  установить SJ1 SJ2 S3
 Для 16 удалить установить SJ4</text>
@@
 <attribute name="VALUE" x="44.45" y="105.918" size="1.778" layer="96"/>
 </instance>
-<instance part="C4" gate="C$" x="35.56" y="99.06"/>
+<instance part="C4" gate="C$" x="35.56" y="99.06" rot="MR0"/>
 <instance part="R4" gate="G$1" x="35.56" y="109.22" smashed="yes" rot="R90">
-<attribute name="NAME" x="34.29" y="117.8814" size="1.778" layer="95" rot="R180"/>
-<attribute name="VALUE" x="34.29" y="115.062" size="1.778" layer="96" rot="R180"/>
+<attribute name="NAME" x="34.29" y="115.3414" size="1.778" layer="95" rot="R180"/>
+<attribute name="VALUE" x="34.29" y="112.522" size="1.778" layer="96" rot="R180"/>
 </instance>
 <instance part="R3" gate="G$1" x="27.94" y="109.22" smashed="yes" rot="R90">

Commit message: rel 1
Parts:
- VT2: device transistor:-NPN-TO220V -> m_transistor:BJT_NPN_TO220_V_BCE
- VT3, VT4: device woofer:-PNP-TO126V -> m_transistor:BJT_PNP_TO126_V_ECB
Connections:
- net CO: now also SJ3.2; no longer SJ2.2
- net N$1: now also R10.A; no longer R10.E
- net N$35: now also SJ3.1; no longer SJ2.1
- net N$37: now also SJ4.2; no longer SJ1.2
- net N$40: now also SJ2.1; no longer SJ3.1
- net N$6: now also R10.E; no longer R10.A
- net N$8: now also SJ1.1; no longer SJ4.1
- net VC+: now also SJ1.2, SJ2.2; no longer SJ3.2, SJ4.2
- net VC-: now also SJ4.1; no longer SJ1.1
Other:
- note added: "L1 PCB"
- note added: "Для 8 установить только SJ2 SJ3 SJ4 Для 16 установить только SJ1"
- note removed: "Для 8 установить SJ1 SJ2 S3 Для 16 удалить установить SJ4"
- moved on the sheet: DA1B, R10, SJ1, SJ2, SJ3, SJ4
